Commit message: mujoco does not support the .dae geometry

File: create_description/urdf/create_2.urdf.xacro (robot description, xacro)
@@ -4,5 +4,5 @@
   <xacro:include filename="$(find create_description)/urdf/create_2_gazebo.urdf.xacro" />
   <xacro:create_base wheel_separation="0.235" base_diameter="0.3485">
-    <mesh filename="package://create_description/meshes/create_2.dae" />
+    <mesh filename="package://create_description/meshes/create_2.stl" />
   </xacro:create_base>
 </robot>

Commit message: improved castor support for the mujoco

File: create_description/urdf/create_2.urdf.xacro (robot description, xacro)
@@ -2,5 +2,4 @@
 <robot name="create_2" xmlns:xacro="http://ros.org/wiki/xacro">
   <xacro:include filename="$(find create_description)/urdf/create_base.urdf.xacro" />
-  <xacro:include filename="$(find create_description)/urdf/create_2_gazebo.urdf.xacro" />
   <xacro:create_base wheel_separation="0.235" base_diameter="0.3485">
     <mesh filename="package://create_description/meshes/create_2.stl" />

File: create_description/urdf/create_base.urdf.xacro (robot description, xacro)
@@ -135,30 +135,4 @@
     <xacro:create_wheel prefix="left" y_offset="${wheel_separation / 2}" wheel_radius="${wheel_radius}" wheel_width="${wheel_width}"/>
     <xacro:create_wheel prefix="right" y_offset="${wheel_separation / -2}" wheel_radius="${wheel_radius}" wheel_width="${wheel_width}"/>
-    <!--<link name="rear_wheel_link">
-    <inertial>
-      <origin xyz="0 0 0"/>
-      <mass value="0.001" />
-      <inertia ixx="0.0001" ixy="0.0" ixz="0.0"
-        iyy="0.0001" iyz="0.0" izz="0.0001" />
-    </inertial>
-    <visual>
-      <origin xyz="0 0 0" rpy="0 ${PI/2} ${PI/2}"/>
-      <geometry>
-        <sphere radius="0.015" />
-      </geometry>
-    </visual>
-    <collision>
-      <origin xyz="0 0 0" rpy="0 ${PI/2} ${PI/2}" />
-      <geometry>
-        <sphere radius="0.015" />
-      </geometry>
-    </collision>
-    </link>
-    <joint name="rear_castor_joint" type="fixed">
-      <origin xyz="-0.13 0 0.0" rpy="0 0 0"/>
-      <parent link="base_link"/>
-      <child link="rear_wheel_link"/>
-      <axis xyz="0 1 0"/>
-    </joint>-->
     <link name="front_wheel_link">
     <inertial>
@@ -180,8 +154,20 @@
     </collision>
     </link>
-    <!-- fixed because there's no transmission -->
-    <joint name="front_castor_joint" type="fixed">
+    <link name="front_turn_link">
+    <inertial>
+      <origin xyz="0 0 0" />
+      <mass value="0.01" />
+      <inertia ixx="0.001" ixy="0.0" ixz="0.0" iyy="0.001" iyz="0.0" izz="0.001" />
+    </inertial>
+    </link>
+    <joint name="front_castor_joint" type="continuous">
       <origin xyz="0.13 0 0.0" rpy="0 0 0" />
       <parent link="base_link" />
+      <child link="front_turn_link" />
+      <axis xyz="1 0 0" />
+    </joint>
+    <joint name="front_wheel_joint" type="continuous">
+      <origin xyz="0 0 0.0" rpy="0 0 0" />
+      <parent link="front_turn_link" />
       <child link="front_wheel_link" />
       <axis xyz="0 1 0" />
@@ -200,13 +186,4 @@
     </inertial>
     </link>
-    <!--
-        TODO (Dmitrii):
-        - Add support for the Mujoco sensors
-    -->
-    <!-- Simulation sensors
-    <xacro:sim_create_base/>
-    <xacro:sim_create_wall_sensor/>
-    <xacro:sim_create_cliff_sensors/>
-    <xacro:sim_imu/> -->
   </xacro:macro>
 </robot>
