Commit message: can be converted to a mujoco model

File: create_description/urdf/create_base.urdf.xacro (robot description, xacro)
@@ -53,5 +53,5 @@
       <mass value="2" />
       <origin xyz="0 0 0.0" />
-      <inertia ixx="0.01" ixy="0.0" ixz="0.0" iyy="0.01" iyz="0.0" izz="0.5" />
+      <inertia ixx="0.024898546" ixy="0.0" ixz="0.0" iyy="0.024898546" iyz="0.0" izz="0.047614879" />
     </inertial>
     <visual>
@@ -93,5 +93,5 @@
       <mass value="0.01" />
       <origin xyz="0 0 0" />
-      <inertia ixx="1.0" ixy="0.0" ixz="0.0" iyy="0.01" iyz="0.0" izz="0.01" />
+      <inertia ixx="0.001" ixy="0.0" ixz="0.0" iyy="0.001" iyz="0.0" izz="0.001" />
     </inertial>
     </link>
@@ -200,9 +200,13 @@
     </inertial>
     </link>
-    <!-- Simulation sensors -->
+    <!--
+        TODO (Dmitrii):
+        - Add support for the Mujoco sensors
+    -->
+    <!-- Simulation sensors
     <xacro:sim_create_base/>
     <xacro:sim_create_wall_sensor/>
     <xacro:sim_create_cliff_sensors/>
-    <xacro:sim_imu/>
+    <xacro:sim_imu/> -->
   </xacro:macro>
 </robot>

Commit message: updated to match the roomba600

File: create_description/urdf/create_base.urdf.xacro (robot description, xacro)
@@ -26,5 +26,5 @@
     </link>
    <joint name="${prefix}_wheel_joint" type="continuous">
-      <origin xyz="0 ${y_offset} 0.015" rpy="0 0 0" />
+      <origin xyz="0 ${y_offset} 0.019" rpy="0 0 0" />
       <parent link="base_link" />
       <child link="${prefix}_wheel_link" />
@@ -56,5 +56,5 @@
     </inertial>
     <visual>
-      <origin xyz=" 0 0 0.0308" rpy="0 0 0" />
+      <origin xyz=" 0 0 0.0201" rpy="0 0 0" />
       <geometry>
         <xacro:insert_block name="mesh" />
@@ -62,5 +62,5 @@
     </visual>
     <collision>
-      <origin xyz="0.0 0.0 0.0308" rpy="0 0 0" />
+      <origin xyz="0.0 0.0 0.0201" rpy="0 0 0" />
       <geometry>
         <cylinder length="0.0611632" radius="0.16495" />

Commit message: fixed joints needed for the teeleoperation

File: create_description/urdf/create_base.urdf.xacro (robot description, xacro)
@@ -135,9 +135,19 @@
     <xacro:create_wheel prefix="left" y_offset="${wheel_separation / 2}" wheel_radius="${wheel_radius}" wheel_width="${wheel_width}"/>
     <xacro:create_wheel prefix="right" y_offset="${wheel_separation / -2}" wheel_radius="${wheel_radius}" wheel_width="${wheel_width}"/>
+    <!-- Intermediate massless body needed for 2-DOF ball-caster approximation -->
+    <link name="front_turn_link">
+    <inertial>
+      <origin xyz="0 0 0" />
+      <mass value="0.0001" />
+      <!-- I = 2/5 * m * r^2 for solid sphere r=0.018: ~1.3e-8; use 1e-7 for stability -->
+      <inertia ixx="0.0000001" ixy="0.0" ixz="0.0" iyy="0.0000001" iyz="0.0" izz="0.0000001" />
+    </inertial>
+    </link>
     <link name="front_wheel_link">
     <inertial>
       <origin xyz="0 0 0" />
-      <mass value="0.01" />
-      <inertia ixx="0.001" ixy="0.0" ixz="0.0" iyy="0.001" iyz="0.0" izz="0.001" />
+      <mass value="0.0001" />
+      <!-- I = 2/5 * m * r^2 for solid sphere r=0.018: ~1.3e-8; use 1e-7 for stability -->
+      <inertia ixx="0.0000001" ixy="0.0" ixz="0.0" iyy="0.0000001" iyz="0.0" izz="0.0000001" />
     </inertial>
     <visual>
@@ -148,5 +158,5 @@
     </visual>
     <collision>
-      <origin xyz="0 0 0" rpy="0 ${PI/2} ${PI/2}" />
+      <origin xyz="0 0 0" rpy="0 0 0" />
       <geometry>
         <sphere radius="0.018" />
@@ -154,16 +164,14 @@
     </collision>
     </link>
-    <link name="front_turn_link">
-    <inertial>
-      <origin xyz="0 0 0" />
-      <mass value="0.01" />
-      <inertia ixx="0.001" ixy="0.0" ixz="0.0" iyy="0.001" iyz="0.0" izz="0.001" />
-    </inertial>
-    </link>
+    <!-- Ball-caster 2-DOF approximation:
+         Joint 1 (Y-axis): forward/backward rolling
+         Joint 2 (X-axis): lateral rolling
+         Together they allow free rolling in any direction, matching an omnidirectional ball caster -->
     <joint name="front_castor_joint" type="continuous">
       <origin xyz="0.13 0 0.0" rpy="0 0 0" />
       <parent link="base_link" />
       <child link="front_turn_link" />
-      <axis xyz="1 0 0" />
+      <axis xyz="0 1 0" />
+      <dynamics damping="0.0" friction="0.0"/>
     </joint>
     <joint name="front_wheel_joint" type="continuous">
@@ -171,5 +179,6 @@
       <parent link="front_turn_link" />
       <child link="front_wheel_link" />
-      <axis xyz="0 1 0" />
+      <axis xyz="1 0 0" />
+      <dynamics damping="0.0" friction="0.0"/>
     </joint>
     <joint name="gyro_joint" type="fixed">
